File: pcb/mimu3000.sch (KiCad schematic (older format))
At the start: 14 parts, among them SW1 P_MISO, SW2 P_MOSI, U1 ATTINY13A-SSU, U2 AQY211EH

Commit message: Switched to attiny48
Parts:
- removed SW1: P_MISO, Connector_PinHeader_2.54mm:PinHeader_1x03_P2.54mm_Vertical, symbol Switch:SW_SPDT
- removed SW2: P_MOSI, Connector_PinHeader_2.54mm:PinHeader_1x03_P2.54mm_Vertical, symbol Switch:SW_SPDT
- added SW1: ONOFF, Pin_Headers:Pin_Header_Straight_1x02_Pitch2.54mm, symbol Switch:SW_DPST_x2
- BT1: footprint Battery:BatteryHolder_Keystone_2468_2xAAA -> Battery_Holders:Keystone_2468_2xAAA
- R1: value 100R -> 580R
- U2: renamed from U1; value ATTINY13A-SSU -> ATTINY48U; footprint Package_SO:SOIC-8_3.9x4.9mm_P1.27mm -> Housings_QFP:TQFP-32_7x7mm_Pitch0.8mm; symbol mimu3000-rescue:ATTINY13A-SSU -> MCU_Microchip_ATtiny:ATtiny48-AU
- renumbered U2 to U1
Connections:
- net labels added: +3V0, GND, LED, MUTE, POT
- wire segments 76 -> 52
Other:
- moved on the sheet: BT1, C1, D1, INPUT1, ISP1, OUTPUT1, R1, R2, RV1, SENS1, U1
