File: pcb/mimu3000.sch (KiCad schematic (older format))
At the start: 19 parts, among them J1 OPT, SW1 ONOFF, SW2 SW_DPDT_x2, U1 AQY211EH, U2 ATTINY88AU

Commit message: Fixed wrong-sized pitch of sensor, corrected witdh of a track. easier footprint for opto
Parts:
- SENS1: footprint Connector_PinHeader_2.00mm:PinHeader_1x04_P2.00mm_Horizontal -> Connector_PinHeader_2.54mm:PinHeader_1x04_P2.54mm_Horizontal
- U1: footprint Package_DIP:DIP-4_W7.62mm -> custom:DIP-4_bubble_W7.62mm
Changed lines of the file:
@@
 F 0 "SENS1" H 6268 2725 50  0000 C CNN
 F 1 "Sens" H 6268 2816 50  0000 C CNN
-F 2 "Connector_PinHeader_2.00mm:PinHeader_1x04_P2.00mm_Horizontal" H 6350 3150 50  0001 C CNN
+F 2 "Connector_PinHeader_2.54mm:PinHeader_1x04_P2.54mm_Horizontal" H 6350 3150 50  0001 C CNN
 F 3 "~" H 6350 3150 50  0001 C CNN
 	1    6350 3150
@@
 F 0 "U1" H 4350 2900 50  0000 L CNN
 F 1 "AQY211EH" H 4350 2800 50  0000 L CNN
-F 2 "Package_DIP:DIP-4_W7.62mm" H 4250 2550 50  0001 C CNN
+F 2 "custom:DIP-4_bubble_W7.62mm" H 4250 2550 50  0001 C CNN
 F 3 "doc/semi_eng_ge1a_aqy21_e.pdf" H 4250 2550 50  0001 C CNN
 	1    4300 2550

Commit message: Fixed misconception that a Capacitor before Opto would smooth the curve
Parts:
- removed C1: 47µ, Capacitor_THT:CP_Radial_D5.0mm_P2.50mm, symbol Device:CP
- removed C5: 1000uF, Capacitor_THT:CP_Radial_D8.0mm_P3.50mm, symbol Device:CP
- added C1: 1uF, Capacitors_THT:C_Rect_L7.0mm_W2.0mm_P5.00mm, symbol Device:C
- C4: value 1000uF -> 1uF; footprint Capacitor_THT:CP_Radial_D8.0mm_P3.50mm -> Capacitors_THT:C_Rect_L7.0mm_W2.0mm_P5.00mm; symbol Device:CP -> Device:C
- RV1: footprint custom:Potentiometer_Generic_5mm_Single_Horizontal -> Potentiometers:Potentiometer_Bourns_PTV09A-2_Vertical
Connections:
- net at C4.1, INPUT1.2, OUTPUT1.2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: now also C1.1
- net at R1.2: now also U1.1
- net at C4.2, SW2.3 (C): now also C1.2
Changed lines of the file:
@@
 	1    0    0    -1
 $EndComp
-$Comp
-L Device:CP C1
-U 1 1 5E2AE194
-P 3950 2100
-F 0 "C1" H 4068 2146 50  0000 L CNN
-F 1 "47µ" H 4068 2055 50  0000 L CNN
-F 2 "Capacitor_THT:CP_Radial_D5.0mm_P2.50mm" H 3988 1950 50  0001 C CNN
-F 3 "~" H 3950 2100 50  0001 C CNN
-	1    3950 2100
-	1    0    0    -1
-$EndComp
-Wire Wire Line
-	3950 2250 3950 2450
 Wire Wire Line
 	3950 2450 4000 2450
@@
 F 0 "RV1" H 3631 5496 50  0000 R CNN
 F 1 "1K_POT" H 3631 5405 50  0000 R CNN
-F 2 "custom:Potentiometer_Generic_5mm_Single_Horizontal" H 3700 5450 50  0001 C CNN
+F 2 "Potentiometers:Potentiometer_Bourns_PTV09A-2_Vertical" H 3700 5450 50  0001 C CNN
 F 3 "~" H 3700 5450 50  0001 C CNN
 	1    3700 5450
@@
 Connection ~ 5500 2750
 $Comp
-L Device:CP C4
+L Device:C C4
 U 1 1 5E4B8635
 P 5500 2900
 F 0 "C4" H 5600 2950 50  0000 L CNN
-F 1 "1000uF" H 5350 2650 50  0000 L CNN
-F 2 "Capacitor_THT:CP_Radial_D8.0mm_P3.50mm" H 5538 2750 50  0001 C CNN
+F 1 "1uF" H 5350 2650 50  0000 L CNN
+F 2 "Capacitors_THT:C_Rect_L7.0mm_W2.0mm_P5.00mm" H 5538 2750 50  0001 C CNN
 F 3 "~" H 5500 2900 50  0001 C CNN
 	1    5500 2900
@@
 Wire Wire Line
 	4300 5150 4300 5300
-$Comp
-L Device:CP C5
-U 1 1 5E4AE3C7
+Wire Wire Line
+	6650 3250 6550 3250
+Wire Wire Line
+	6650 2700 6650 3250
+Wire Wire Line
+	6750 3400 6750 3150
+Wire Wire Line
+	6750 3150 6550 3150
+Wire Wire Line
+	6550 3050 6850 3050
+Wire Wire Line
+	6850 2950 6550 2950
+Wire Wire Line
+	3950 1950 3950 2450
+$Comp
+L Device:C C1
+U 1 1 5E688126
 P 5800 2900
-F 0 "C5" H 5600 2850 50  0000 L CNN
-F 1 "1000uF" H 5650 3150 50  0000 L CNN
-F 2 "Capacitor_THT:CP_Radial_D8.0mm_P3.50mm" H 5838 2750 50  0001 C CNN
+F 0 "C1" H 5900 2950 50  0000 L CNN
+F 1 "1uF" H 5650 2650 50  0000 L CNN
+F 2 "Capacitors_THT:C_Rect_L7.0mm_W2.0mm_P5.00mm" H 5838 2750 50  0001 C CNN
 F 3 "~" H 5800 2900 50  0001 C CNN
 	1    5800 2900
-	-1   0    0    1
+	1    0    0    -1
 $EndComp
 Wire Wire Line
@@
 	5500 3050 5800 3050
 Connection ~ 5500 3050
-Wire Wire Line
-	6650 3250 6550 3250
-Wire Wire Line
-	6650 2700 6650 3250
-Wire Wire Line
-	6750 3400 6750 3150
-Wire Wire Line
-	6750 3150 6550 3150
-Wire Wire Line
-	6550 3050 6850 3050
-Wire Wire Line
-	6850 2950 6550 2950
 $EndSCHEMATC
