File: pcb/mimu_batt.sch (KiCad schematic (older format))
At the start: 2 parts, among them SW1 ONOFF

Commit message: I hope this did not break everything
Connections:
- net labels added: VCC
- net labels removed: +3V0
Changed lines of the file:
@@
-$EndComp
-$Comp
-L power:+3V0 #PWR01
-U 1 1 5E41CB28
-P 2450 2600
-F 0 "#PWR01" H 2450 2450 50  0001 C CNN
-F 1 "+3V0" H 2465 2773 50  0000 C CNN
-F 2 "" H 2450 2600 50  0001 C CNN
-F 3 "" H 2450 2600 50  0001 C CNN
-	1    2450 2600
-	1    0    0    -1
 $EndComp
 $Comp
@@
 F1 "mimu_base.sch" 50
 $EndSheet
+$Comp
+L power:VCC #PWR0101
+U 1 1 5E6A4AB9
+P 2450 2600
+F 0 "#PWR0101" H 2450 2450 50  0001 C CNN
+F 1 "VCC" H 2467 2773 50  0000 C CNN
+F 2 "" H 2450 2600 50  0001 C CNN
+F 3 "" H 2450 2600 50  0001 C CNN
+	1    2450 2600
+	1    0    0    -1
+$EndComp
 $EndSCHEMATC
