File: pcb/mimu_base.sch (KiCad schematic (older format))
At the start: 16 parts, among them J1 OPT, SW2 SW_DPDT_x2, U1 AQY211EH, U2 ATTINY88AU

Commit message: I hope this did not break everything
Parts:
- C3, C4: footprint Capacitors_THT:C_Rect_L7.0mm_W2.0mm_P5.00mm -> Capacitor_THT:C_Rect_L7.0mm_W3.5mm_P2.50mm_P5.00mm
- R1, R2: footprint Resistor_THT:R_Axial_DIN0207_L6.3mm_D2.5mm_P7.62mm_Horizontal -> Resistor_SMD:R_1206_3216Metric_Pad1.42x1.75mm_HandSolder
- RV1: footprint Potentiometers:Potentiometer_Bourns_PTV09A-2_Vertical -> Potentiometer_THT:Potentiometer_Bourns_PTV09A-2_Single_Horizontal
- renumbered D1 to D_LED1
Connections:
- net +3V0: no longer C1.1, C2.1, J1.5 (Pin_5), RV1.3, SENS1.1 (VCC), U2.18 (AVCC), U2.4 (VCC)
- new net VCC: C1.1, C2.1, J1.5 (Pin_5), RV1.3, SENS1.1 (VCC), U2.18 (AVCC), U2.4 (VCC)
Other:
- moved on the sheet: C2

Commit message: Quick layout test
Connections:
- net XLR_COLD: now reaches INPUT1.3, OUTPUT1.3, U1.4
- net XLR_GND: now reaches INPUT1.1, OUTPUT1.1
- net XLR_HOT: now reaches C3.1, C4.1, INPUT1.2, OUTPUT1.2, SW2.1 (A)
Changed lines of the file:
@@
 	4850 2250 4800 2250
 Wire Wire Line
-	5500 1450 5500 2250
-Wire Wire Line
-	4800 1450 4800 2250
+	5500 1450 5500 1700
+Wire Wire Line
+	4800 1450 4800 1850
 Wire Wire Line
 	5150 1850 5650 1850
@@
 Wire Wire Line
 	7650 3900 7650 3950
+Text GLabel 6000 1600 1    50   Input ~ 0
+XLR_HOT
+Text GLabel 6200 1600 1    50   Input ~ 0
+XLR_COLD
+Text GLabel 4550 1800 1    50   Input ~ 0
+XLR_GND
+Wire Wire Line
+	4550 1800 4550 1850
+Wire Wire Line
+	4550 1850 4800 1850
+Connection ~ 4800 1850
+Wire Wire Line
+	4800 1850 4800 2250
+Wire Wire Line
+	6000 1600 6000 1700
+Wire Wire Line
+	6000 1700 5500 1700
+Connection ~ 5500 1700
+Wire Wire Line
+	5500 1700 5500 2250
+Wire Wire Line
+	6200 1600 6200 1850
+Wire Wire Line
+	6200 1850 5650 1850
+Connection ~ 5650 1850
 $EndSCHEMATC

Commit message: Now it just has to work, lol
Parts:
- added TP5: TestPoint, Measurement_Points:Measurement_Point_Round-SMD-Pad_Small, symbol Connector:TestPoint
Connections:
- net POT: now also TP5.1
Changed lines of the file:
@@
 POT
 Wire Wire Line
-	3550 5600 3300 5600
+	3550 5600 3400 5600
 Text GLabel 3300 5600 0    50   Input ~ 0
 POT
@@
 	6200 1850 5650 1850
 Connection ~ 5650 1850
+$Comp
+L Connector:TestPoint TP5
+U 1 1 5E6DA51D
+P 3400 5600
+F 0 "TP5" H 3250 5900 50  0000 L CNN
+F 1 "TestPoint" H 3250 5800 50  0000 L CNN
+F 2 "Measurement_Points:Measurement_Point_Round-SMD-Pad_Small" H 3600 5600 50  0001 C CNN
+F 3 "~" H 3600 5600 50  0001 C CNN
+	1    3400 5600
+	1    0    0    -1
+$EndComp
+Connection ~ 3400 5600
+Wire Wire Line
+	3400 5600 3300 5600
 $EndSCHEMATC

Commit message: Buy all the shit
Parts:
- removed C4: 1uF, Capacitor_THT:C_Rect_L7.0mm_W3.5mm_P2.50mm_P5.00mm, symbol Device:C
Changed lines of the file:
@@
 Comment4 ""
 $EndDescr
-Connection ~ 5500 3200
-Wire Wire Line
-	5500 3200 5800 3200
-Wire Wire Line
-	5800 2900 5500 2900
-$Comp
-L Device:C C4
-U 1 1 5E6D36B1
-P 5800 3050
-F 0 "C4" H 5900 3100 50  0000 L CNN
-F 1 "1uF" H 5650 2800 50  0000 L CNN
-F 2 "Capacitor_THT:C_Rect_L7.0mm_W3.5mm_P2.50mm_P5.00mm" H 5838 2900 50  0001 C CNN
-F 3 "~" H 5800 3050 50  0001 C CNN
-	1    5800 3050
-	1    0    0    -1
-$EndComp
 Wire Wire Line
 	3950 2100 3950 2600
