File: pcb/mimu_batt.kicad_pcb (KiCad board)
At the start: 2 copper layers, 54.8 x 40 mm, 19 parts, among them J1 OPT, SW1 ONOFF, SW2 SW_DPDT_x2, U1 AQY211EH, U2 ATTINY88AU

Commit message: divided schematics to hierarchically have battery and phantom powered variant
Parts:
- removed C5: 1000uF, Capacitor_THT:CP_Radial_D8.0mm_P3.50mm
- C1: value 47µ -> 1uF; footprint Capacitor_THT:CP_Radial_D5.0mm_P2.50mm -> Capacitors_THT:C_Rect_L7.0mm_W2.0mm_P5.00mm
- C4: value 1000uF -> 1uF; footprint Capacitor_THT:CP_Radial_D8.0mm_P3.50mm -> Capacitors_THT:C_Rect_L7.0mm_W2.0mm_P5.00mm
- RV1: footprint custom:Potentiometer_Generic_5mm_Single_Horizontal -> Potentiometers:Potentiometer_Bourns_PTV09A-2_Vertical
- moved C1 26.5 mm to (207.8, 123.2), turned to 90 degrees
- moved RV1 6.17 mm to (175.2, 94.0)
- moved C4 5.33 mm to (204.5, 123.2)
- moved INPUT1 1.40 mm to (196.5, 123.8)
- moved OUTPUT1 1.25 mm to (214.8, 123.8)
Connections:
- C4 pad 1: Net-(C4-Pad1) -> Net-(C1-Pad1)
- C4 pad 2: Net-(C4-Pad2) -> Net-(C1-Pad2)
- INPUT1 pad 2: Net-(C4-Pad1) -> Net-(C1-Pad1)
- OUTPUT1 pad 2: Net-(C4-Pad1) -> Net-(C1-Pad1)
- R1 pad 2: Net-(C1-Pad1) -> Net-(R1-Pad2)
- SW2 pad 1: Net-(C4-Pad1) -> Net-(C1-Pad1)
- SW2 pad 3: Net-(C4-Pad2) -> Net-(C1-Pad2)
- U1 pad 1: Net-(C1-Pad2) -> Net-(R1-Pad2)
- U2 pad 1: (no net) -> Net-(U2-Pad1)
- U2 pad 10: (no net) -> Net-(U2-Pad10)
- U2 pad 11: (no net) -> Net-(U2-Pad11)
- U2 pad 12: (no net) -> Net-(U2-Pad12)
- U2 pad 13: (no net) -> Net-(U2-Pad13)
- U2 pad 14: (no net) -> Net-(U2-Pad14)
- U2 pad 19: (no net) -> Net-(U2-Pad19)
- U2 pad 2: (no net) -> Net-(U2-Pad2)
- U2 pad 20: (no net) -> Net-(U2-Pad20)
- U2 pad 22: (no net) -> Net-(U2-Pad22)
- U2 pad 26: (no net) -> Net-(U2-Pad26)
- U2 pad 3: (no net) -> Net-(U2-Pad3)
- U2 pad 6: (no net) -> Net-(U2-Pad6)
- U2 pad 7: (no net) -> Net-(U2-Pad7)
- U2 pad 8: (no net) -> Net-(U2-Pad8)
- U2 pad 9: (no net) -> Net-(U2-Pad9)
Routing:
- net Net-(R1-Pad2): track 0.00 -> 32.6 mm
- net Net-(C4-Pad1): track 30.5 -> 0.00 mm
- net Net-(C1-Pad1): track 3.12 -> 28.0 mm
- net Net-(C1-Pad2): track 27.0 -> 10.1 mm
- net Net-(C4-Pad2): track 13.7 -> 0.00 mm
- net GND: track 175.0 -> 164.4 mm
- net +3V0: track 130.7 -> 127.4 mm
- net Net-(INPUT1-Pad1): track 21.8 -> 19.2 mm
- net Net-(INPUT1-Pad3): track 24.4 -> 22.5 mm
- net POT: track 23.0 -> 21.3 mm, vias 1 -> 2
Other:
- board text added: "MIMU Batt v0.6 PP 03.19"
- board text removed: "MIMU3000 v0.5 PP 03.19"

Commit message: Bump near-final version for battery powered version. Todo: Maybe remove the capacitor? Needs realworld-test.
Parts:
- moved SW1 9.32 mm to (167.6, 122.6), turned to 180 degrees
- moved BT1 0.22 mm to (167.6, 119.8)
Connections:
- SW1 pad 1: +3V0 -> VCC
Routing:
- net +3V0: track 127.4 -> 126.5 mm
Other:
- board text added: "MIMU Batt v0.7 PP 03.20"
- board text removed: "MIMU Batt v0.6 PP 03.19"

Commit message: Quick order of some pcbs
Other:
- board text added: "https://github.com/Cirromulus/mimu"
Changed lines of the file:
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@@
   (general
     (thickness 1.6)
-    (drawings 35)
+    (drawings 36)
     (tracks 209)
     (zones 0)
@@
       (drillshape 0)
       (scaleselection 1)
-      (outputdirectory "gerber/"))
+      (outputdirectory "gerber/mimu_batt"))
   )
   (net 0 "")
@@
     )
   )
-  (gr_text JLCJLCJLCJLC (at 172.4 99.4 180) (layer B.SilkS)
+  (gr_text https://github.com/Cirromulus/mimu (at 191.6 92) (layer B.SilkS)
     (effects (font (size 1 1) (thickness 0.15)) (justify mirror))
   )
-  (gr_text lol (at 172.4 100.9) (layer B.SilkS)
+  (gr_text JLCJLCJLCJLC (at 191.2 114.8 180) (layer B.SilkS)
+    (effects (font (size 1 1) (thickness 0.15)) (justify mirror))
+  )
+  (gr_text lol (at 191.2 116.3) (layer B.SilkS)
     (effects (font (size 1 1) (thickness 0.15)) (justify mirror))
   )
@@
     (effects (font (size 1 1) (thickness 0.15)))
   )
-  (gr_text CLD (at 216.093 118.818) (layer F.SilkS)
+  (gr_text CLD (at 216.293 118.818) (layer F.SilkS)
     (effects (font (size 0.5 0.5) (thickness 0.1)) (justify left))
   )
-  (gr_text HOT (at 216.093 121.358) (layer F.SilkS)
+  (gr_text HOT (at 216.293 121.358) (layer F.SilkS)
     (effects (font (size 0.5 0.5) (thickness 0.1)) (justify left))
   )
-  (gr_text GND (at 216.093 123.898) (layer F.SilkS)
+  (gr_text GND (at 216.293 123.898) (layer F.SilkS)
     (effects (font (size 0.5 0.5) (thickness 0.1)) (justify left))
   )
