File: pcb/mimu_phantom.kicad_sch (KiCad schematic)
At the start: 18 parts, among them U3 MCP16331CH

Commit message: First layout
Parts:
- added C3: 50-100uF, Capacitor_THT:CP_Radial_D4.0mm_P2.00mm, symbol Device:C_Polarized
- C_pre1, C_pre2: value 50-100uF @24V -> 3-4uF @24V
- R3, R4: footprint Resistor_SMD:R_0805_2012Metric_Pad1.20x1.40mm_HandSolder -> Resistor_SMD:R_1206_3216Metric_Pad1.30x1.75mm_HandSolder
Connections:
- net +BATT: now also C_pre2.1
- net GND: now also C_pre1.2, C3.2
- net VCC: now also C3.1
Other:
- moved on the sheet: C_pre1

Commit message: Minor PCB updates
Parts:
- C3: footprint Capacitor_THT:CP_Radial_D4.0mm_P2.00mm -> Capacitor_THT:CP_Radial_D5.0mm_P2.00mm
- C_IN1, C_IN2: value 10uF -> 10uF @ 24v
Changed lines of the file:
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@@
   (symbol (lib_id "Device:C") (at 41.91 129.54 0) (unit 1)
     (in_bom yes) (on_board yes)
-    (property "Reference" "C_IN1" (id 0) (at 44.831 128.3716 0)
-      (effects (font (size 1.27 1.27)) (justify left))
-    )
-    (property "Value" "10uF" (id 1) (at 44.831 130.683 0)
+    (property "Reference" "C_IN1" (id 0) (at 27.94 128.4986 0)
+      (effects (font (size 1.27 1.27)) (justify left))
+    )
+    (property "Value" "10uF @ 24v" (id 1) (at 27.94 130.81 0)
       (effects (font (size 1.27 1.27)) (justify left))
     )
@@
       (effects (font (size 1.27 1.27)) (justify left))
     )
-    (property "Value" "10uF" (id 1) (at 56.261 130.683 0)
+    (property "Value" "10uF @ 24v" (id 1) (at 56.261 130.683 0)
       (effects (font (size 1.27 1.27)) (justify left))
     )
@@
     )
     (property "Value" "50-100uF" (id 1) (at 152.781 135.4332 0)
-      (effects (font (size 1.27 1.27)) (justify left) hide)
-    )
-    (property "Footprint" "Capacitor_THT:CP_Radial_D4.0mm_P2.00mm" (id 2) (at 150.8252 138.43 0)
-      (effects (font (size 1.27 1.27)) hide)
-    )
-    (property "Datasheet" "~" (id 3) (at 149.86 134.62 0)
+      (effects (font (size 1.27 1.27)) (justify left))
+    )
+    (property "Footprint" "Capacitor_THT:CP_Radial_D5.0mm_P2.00mm" (id 2) (at 150.8252 138.43 0)
+      (effects (font (size 1.27 1.27)) hide)
+    )
+    (property "Datasheet" "https://www.digikey.de/de/products/detail/rubycon/6-3MS7100MEFCTZ5X7/3566526" (id 3) (at 149.86 134.62 0)
       (effects (font (size 1.27 1.27)) hide)
     )
@@
     )
     (path "/108fa6a7-bc8c-478f-94da-d7d6f62a48b1"
-      (reference "C3") (unit 1) (value "50-100uF") (footprint "Capacitor_THT:CP_Radial_D4.0mm_P2.00mm")
+      (reference "C3") (unit 1) (value "50-100uF") (footprint "Capacitor_THT:CP_Radial_D5.0mm_P2.00mm")
     )
     (path "/00000000-0000-0000-0000-00005e6a72eb"
@@
     )
     (path "/00000000-0000-0000-0000-00005e6a4eb3"
-      (reference "C_IN1") (unit 1) (value "10uF") (footprint "Capacitor_SMD:C_1206_3216Metric_Pad1.42x1.75mm_HandSolder")
+      (reference "C_IN1") (unit 1) (value "10uF @ 24v") (footprint "Capacitor_SMD:C_1206_3216Metric_Pad1.42x1.75mm_HandSolder")
     )
     (path "/00000000-0000-0000-0000-00005e6a593e"
-      (reference "C_IN2") (unit 1) (value "10uF") (footprint "Capacitor_SMD:C_1206_3216Metric_Pad1.42x1.75mm_HandSolder")
+      (reference "C_IN2") (unit 1) (value "10uF @ 24v") (footprint "Capacitor_SMD:C_1206_3216Metric_Pad1.42x1.75mm_HandSolder")
     )
     (path "/00000000-0000-0000-0000-00005e6a672d"

Commit message: Small cleanups
Parts:
- C_IN1, C_IN2: value 10uF @ 24v -> 10uF @ 48v
- C_pre1: value 3-4uF @24V -> 3-4uF @48V
- C_pre2: value 3-4uF @24V -> 3-4uF @48v
Changed lines of the file:
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@@
 			)
 		)
-		(property "Value" "10uF @ 24v"
+		(property "Value" "10uF @ 48v"
 			(at 27.94 130.81 0)
 			(effects
@@
 			)
 		)
-		(property "Value" "10uF @ 24v"
+		(property "Value" "10uF @ 48v"
 			(at 56.261 130.683 0)
 			(effects
@@
 			)
 		)
-		(property "Value" "3-4uF @24V"
+		(property "Value" "3-4uF @48V"
 			(at 58.42 73.66 0)
 			(effects
@@
 			)
 		)
-		(property "Value" "3-4uF @24V"
+		(property "Value" "3-4uF @48v"
 			(at 33.02 73.66 0)
 			(effects

Commit message: Some goof-arounds, but real prototype still produces wobbles with sensor current draw
Parts:
- added C_Top: 20pF, Capacitor_SMD:C_1206_3216Metric_Pad1.42x1.75mm_HandSolder, symbol Device:C
- C3: value 50-100uF -> Optional, 20-50uF
- C_IN1: value 10uF @ 48v -> 4uF @48v (X5R?)
- C_IN2: value 10uF @ 48v -> 100nF @48v
- C_pre1: value 3-4uF @48V -> 4uF @48v (X5R?)
- C_pre2: value 3-4uF @48v -> 100nF @48v
- D1: footprint Diodes_SMD:D_SMA -> Diode_SMD:D_SMA
- R3, R4: value 6.8kOhm 0.1% -> ~4kOhm 0.1%
Connections:
- net VCC: now also C_Top.1
- net at R_BOT1.1, R_TOP1.2, TP4.1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: now also C_Top.2
Other:
- note added: "(Optional)"
- moved on the sheet: C3, R_TOP1

Commit message: Added emphasis on having less VCC. 3v work fine, perhaps even less.
Parts:
- R_TOP1: value 31.2k -> 27.5k - 31.2k
Other:
- note added: "V_FB = 0.8v"
- note added: "V_out = V_s * R_2 / (R_1 + R_2) with V_FB = 0.8v and V_s target ~3v R_top = (R_bot * ( V_s - V_out)) / V_out R_top = (10k * (3v - 0.8v)) / 0.8v R_top = 27.5k"
- note removed: "31.2/10 = 3.12v"
- note removed: "V_FB =~ 1v"
Changed lines of the file:
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@@
 		)
 	)
-	(text "31.2/10 = 3.12v"
-		(exclude_from_sim no)
-		(at 129.54 140.97 90)
+	(text "V_out = V_s * R_2 / (R_1 + R_2)\n\nwith V_FB = 0.8v\nand V_s target ~3v\n\nR_top = (R_bot * ( V_s - V_out)) / V_out\nR_top = (10k * (3v - 0.8v)) / 0.8v\nR_top = 27.5k\n"
+		(exclude_from_sim no)
+		(at 107.188 159.004 0)
 		(effects
 			(font
-				(size 1.27 1.27)
-			)
-			(justify right bottom)
+				(size 0.762 0.762)
+			)
+			(justify left bottom)
 		)
 	)
@@
 		)
 	)
-	(text "V_FB =~ 1v"
+	(text "V_FB = 0.8v"
 		(exclude_from_sim no)
 		(at 87.63 133.35 90)
@@
 			)
 		)
-		(property "Value" "31.2k"
-			(at 136.398 138.303 0)
-			(effects
-				(font
+		(property "Value" "27.5k - 31.2k"
+			(at 127.508 138.176 0)
+			(effects
+				(font
